Commit message: created new launch file for gazebo

File: description/robot_core.xacro (robot description, xacro)
@@ -10,5 +10,5 @@
         <parent link="base_link"/>
         <child link="chassis"/>
-        <origin xyz="-0.1 0 0"/>
+        <origin xyz="-0.1 0 0.025"/>
     </joint>
     <link name="chassis">
